Commit message: Adding pressure sensor / Fixing imu

File: urdf/gazebo.urdf.xacro (robot description, xacro)
@@ -8,5 +8,16 @@
           <topic>imu</topic>
         </sensor>
+    </gazebo>
+    <gazebo reference="$(arg prefix)_pressure">
+        <sensor name="$(arg prefix)_pressure_sensor" type="altimeter">
+            <always_on>1</always_on>
+            <update_rate>100.0</update_rate>
+            <visualize>true</visualize>
+            <topic>/altimeter</topic>
+        </sensor>
+    </gazebo>
+    <gazebo>
         <plugin filename="ignition-gazebo-imu-system" name="ignition::gazebo::systems::Imu" />
+        <plugin filename="ignition-gazebo-altimeter-system" name="ignition::gazebo::systems::Altimeter" />
     </gazebo>
     <gazebo>

File: urdf/riptide.urdf.xacro (robot description, xacro)
@@ -71,4 +71,16 @@
 		<dynamics damping="0.0" friction="0.0"/>
 	</joint>
+	<link name="$(arg prefix)_pressure">
+		<inertial>
+			<mass value="0.001"/>
+			<inertia ixx="0.0000001" ixy="0" ixz="0" iyy="0.0000001" iyz="0" izz="0.0000001"/>
+		</inertial>
+	</link>
+	<joint name="$(arg prefix)_pressure_joint" type="fixed">
+		<origin xyz="0.0 0.0 0.0"/>
+		<parent link="$(arg prefix)"/>
+		<child link="$(arg prefix)_pressure"/>
+		<dynamics damping="0.0" friction="0.0"/>
+	</joint>
 	<xacro:include filename="$(find riptide_description_sim)/urdf/riptide_fin.urdf.xacro"/>
 	<xacro:riptide_fin name="d" orientation="0"/>

Commit message: Adding Thruster plugin, fixing urdf

File: urdf/gazebo.urdf.xacro (robot description, xacro)
@@ -25,25 +25,25 @@
             <parameters>$(find riptide_bringup_sim)/config/riptide_controllers.yaml</parameters>
         </plugin>
-        <plugin filename="ignition-gazebo-thruster-system" name="ignition::gazebo::systems::Thruster">
+        <plugin filename="riptide_plugins" name="riptide_plugins::Thruster">
             <joint_name>$(arg prefix)_thruster_joint</joint_name>
-            <thrust_coefficient>0.004422</thrust_coefficient>
+            <!-- <use_angvel_cmd>true</use_angvel_cmd> -->
             <fluid_density>1000</fluid_density>
             <propeller_diameter>0.1</propeller_diameter>
-            <use_angvel_cmd>true</use_angvel_cmd>
+            <thrust_coefficient>0.0004</thrust_coefficient>
         </plugin>
         <plugin filename="ignition-gazebo-hydrodynamics-system" name="ignition::gazebo::systems::Hydrodynamics">
             <link_name>base_link</link_name> <!-- dummy_link and riptide link are fusionned in gazebo as the joint between the two links is fixed-->
-            <xDotU>-0.01</xDotU>
+            <xDotU>-0.001</xDotU>
             <yDotV>-0.05</yDotV>
             <zDotW>-0.05</zDotW>
-            <kDotP>-0.01</kDotP>
+            <kDotP>-0.001</kDotP>
             <mDotQ>-0.05</mDotQ>
             <nDotR>-0.05</nDotR>
-            <xUabsU>-5</xUabsU>
-            <yVabsV>-1000</yVabsV>
-            <zWabsW>-1000</zWabsW>
-            <kPabsP>-1</kPabsP>
-            <mQabsQ>-700</mQabsQ>
-            <nRabsR>-700</nRabsR>
+            <xUabsU>-0.1</xUabsU>
+            <yVabsV>-10</yVabsV>
+            <zWabsW>-10</zWabsW>
+            <kPabsP>-0.1</kPabsP>
+            <mQabsQ>-100</mQabsQ>
+            <nRabsR>-100</nRabsR>
             <xU>-0.1</xU>
             <yV>-0.1</yV>

File: urdf/riptide.urdf.xacro (robot description, xacro)
@@ -13,5 +13,5 @@
 			<origin xyz="0.12 0 0.08" rpy="${-pi/2} 0 ${pi}"/>
 			<mass value="9"/>
-			<inertia ixx="0.03675" ixy="0" ixz="0" iyy="1.1465" iyz="0" izz="1.1465"/>
+			<inertia ixx="0.03675" ixy="0" ixz="0" iyy="0.8" iyz="0" izz="0.8"/>
 		</inertial>
 		<collision>
@@ -36,5 +36,5 @@
 		</visual>
 		<inertial>
-			<mass value="0.02" />
+			<mass value="0.01" />
 			<inertia ixx="0.00001" ixy="0" ixz="0" iyy="0.00001" iyz="0" izz="0.000005" />
 		</inertial>
@@ -57,5 +57,5 @@
 		<parent link="$(arg prefix)"/>
 		<child link="$(arg prefix)_thruster"/>
-		<dynamics damping="0.0" friction="0.0"/>
+		<dynamics damping="0.00001" friction="0.00001"/>
 	</joint>
 	<link name="$(arg prefix)_imu">

File: urdf/riptide_fin.urdf.xacro (robot description, xacro)
@@ -26,5 +26,5 @@
 			<parent link="$(arg prefix)"/>
 			<child link="$(arg prefix)_${name}_fin"/>
-			<limit effort="1000.0" lower="${-pi/4}" upper="${pi/4}" velocity="0.5"/>
+			<limit effort="10000" lower="${-pi/8}" upper="${pi/8}" velocity="2"/> <!-- velocity = 0.5-->
 			<dynamics damping="0.1" friction="0.1"/>
 		</joint>
@@ -38,10 +38,10 @@
 				<cda>0.2</cda>
 				<cda_stall>0.03</cda_stall>
-				<alpha_stall>0.17</alpha_stall>
+				<alpha_stall>0.4</alpha_stall>
 				<a0>0</a0>
-				<area>0.0244</area>
+				<area>0.05</area>
 				<upward>0 1 0</upward>
 				<forward>1 0 0</forward>
-				<cp>0 0 0.05</cp>
+				<cp>0 0 0</cp>
 			</plugin>
 		</gazebo>

Commit message: Updating coefficients simulation

File: urdf/gazebo.urdf.xacro (robot description, xacro)
@@ -34,22 +34,22 @@
         <plugin filename="ignition-gazebo-hydrodynamics-system" name="ignition::gazebo::systems::Hydrodynamics">
             <link_name>base_link</link_name> <!-- dummy_link and riptide link are fusionned in gazebo as the joint between the two links is fixed-->
-            <xDotU>-0.001</xDotU>
-            <yDotV>-0.05</yDotV>
-            <zDotW>-0.05</zDotW>
-            <kDotP>-0.001</kDotP>
-            <mDotQ>-0.05</mDotQ>
-            <nDotR>-0.05</nDotR>
-            <xUabsU>-0.1</xUabsU>
-            <yVabsV>-10</yVabsV>
-            <zWabsW>-10</zWabsW>
-            <kPabsP>-0.1</kPabsP>
-            <mQabsQ>-100</mQabsQ>
-            <nRabsR>-100</nRabsR>
-            <xU>-5.</xU>
-            <yV>-0.1</yV>
-            <zW>-0.1</zW>
-            <kP>-0.1</kP>
-            <mQ>-0.1</mQ>
-            <nR>-0.1</nR>
+            <xDotU>-7.</xDotU>
+            <yDotV>-0.5</yDotV>
+            <zDotW>-0.5</zDotW>
+            <kDotP>-0.01</kDotP>
+            <mDotQ>-0.1</mDotQ>
+            <nDotR>-0.1</nDotR>
+            <xUabsU>-0.01</xUabsU>
+            <yVabsV>-0.05</yVabsV>
+            <zWabsW>-0.05</zWabsW>
+            <kPabsP>-0.05</kPabsP>
+            <mQabsQ>-0.01</mQabsQ>
+            <nRabsR>-0.01</nRabsR>
+            <xU>-2.</xU>
+            <yV>-5.</yV>
+            <zW>-5.</zW>
+            <kP>-1.</kP>
+            <mQ>-3.</mQ>
+            <nR>-3.</nR>
         </plugin>
     </gazebo>

File: urdf/riptide.urdf.xacro (robot description, xacro)
@@ -11,10 +11,10 @@
 		</visual>
 		<inertial>
-			<origin xyz="0.12 0 0.08" rpy="${-pi/2} 0 ${pi}"/>
+			<origin xyz="0.12 0 0.14" rpy="${-pi/2} 0 ${pi}"/>
 			<mass value="9"/>
 			<inertia ixx="0.03675" ixy="0" ixz="0" iyy="0.8" iyz="0" izz="0.8"/>
 		</inertial>
 		<collision>
-			<origin xyz="0 0 0" rpy="0 ${-pi/2} 0" />
+			<origin xyz="0 0 -0.2" rpy="0 ${-pi/2} 0" />
 			<geometry>
 				<box size="0.12 0.12 0.95" />
@@ -58,4 +58,5 @@
 		<child link="$(arg prefix)_thruster"/>
 		<dynamics damping="0.00001" friction="0.00001"/>
+		<limit effort="1000" velocity="350"/>
 	</joint>
 	<link name="$(arg prefix)_imu">

File: urdf/riptide_fin.urdf.xacro (robot description, xacro)
@@ -15,7 +15,7 @@
             </inertial>
 			<collision>
-				<origin xyz="-0.01 0.04 0" rpy="0 0 0" />
+				<origin xyz="-0.01 0 0.04" rpy="0 0 0" />
                 <geometry>
-                    <box size="0.08 0.1 0.08" />
+                    <box size="0.08 0.01 0.08" />
                 </geometry>
             </collision>
@@ -34,11 +34,11 @@
 				<control_joint_name>$(arg prefix)_${name}_joint</control_joint_name>
 				<air_density>1000</air_density>
-				<cla>4.13</cla>
-				<cla_stall>-1.1</cla_stall>
-				<cda>0.2</cda>
-				<cda_stall>0.03</cda_stall>
-				<alpha_stall>0.4</alpha_stall>
 				<a0>0</a0>
-				<area>0.05</area>
+				<cla>7.16</cla>
+				<cla_stall>-1.5</cla_stall>
+				<cda>0.038</cda>
+				<cda_stall>1.146</cda_stall>
+				<alpha_stall>0.26</alpha_stall>
+				<area>0.005</area>
 				<upward>0 1 0</upward>
 				<forward>1 0 0</forward>
