Commit message: Updating for gazebo simulation

File: urdf/riptide.urdf.xacro (robot description, xacro)
@@ -1,19 +1,31 @@
 <?xml version="1.0"?>
 <robot name="$(arg prefix)" xmlns:xacro="http://www.ros.org/wiki/xacro">
+	<link name="base_link" />
     <!-- Rigid body description of the base link -->
 	<link name="$(arg prefix)">
 		<visual>
-			<origin xyz="0.2 0 0" rpy="${pi/2} 0 ${pi}"/>
+			<origin xyz="0.2 0 0" rpy="${-pi/2} 0 ${pi}"/>
 			<geometry>
 				<mesh filename="package://riptide_description_sim/meshes/riptide_body.stl" scale="0.001 0.001 0.001"/>
 			</geometry>
-		  </visual>
+		</visual>
+		<inertial>
+			<origin xyz="0.12 0 0.08" rpy="${-pi/2} 0 ${pi}"/>
+			<mass value="9"/>
+			<inertia ixx="0.03675" ixy="0" ixz="0" iyy="1.1465" iyz="0" izz="1.1465"/>
+		</inertial>
+		<collision>
+			<origin xyz="0 0 0" rpy="0 ${-pi/2} 0" />
+			<geometry>
+				<box size="0.12 0.12 0.95" />
+			</geometry>
+		</collision>
 	</link>
-	<link name="$(arg prefix)_echosounder"/>
-	<joint name="$(arg prefix)_echosounder" type="fixed">
+	<!-- <link name="$(arg prefix)_echosounder"/> -->
+	<!-- <joint name="$(arg prefix)_echosounder" type="fixed">
 		<origin rpy="0 ${pi/2} 0" xyz="0.28 0 -0.05"/>
 		<parent link="$(arg prefix)"/>
 		<child link="$(arg prefix)_echosounder"/>
-	</joint>
+	</joint> -->
 	<link name="$(arg prefix)_thruster">
 		<visual>
@@ -23,10 +35,39 @@
 			</geometry>
 		</visual>
+		<inertial>
+			<mass value="0.02" />
+			<inertia ixx="0.00001" ixy="0" ixz="0" iyy="0.00001" iyz="0" izz="0.000005" />
+		</inertial>
+		<collision>
+			<origin xyz="0 0 0" rpy="0 ${pi/2} 0"/>
+			<geometry>
+				<cylinder radius="0.04" length="0.03"/>
+			</geometry>
+		</collision>
 	</link>
-	<joint name="$(arg prefix)_thruster" type="continuous">
+	<joint name="$(arg prefix)_base_link" type="fixed">
+		<origin rpy="0 0 0" xyz="-0.51 0 0"/>
+		<parent link="base_link"/>
+		<child link="$(arg prefix)"/>
+		<dynamics damping="0.0" friction="0.0"/>
+	</joint>
+	<joint name="$(arg prefix)_thruster_joint" type="continuous">
 		<axis xyz="1 0 0"/>
 		<origin rpy="0 0 0" xyz="-0.51 0 0"/>
 		<parent link="$(arg prefix)"/>
 		<child link="$(arg prefix)_thruster"/>
+		<dynamics damping="0.0" friction="0.0"/>
+	</joint>
+	<link name="$(arg prefix)_imu">
+		<inertial>
+			<mass value="0.001"/>
+			<inertia ixx="0.0000001" ixy="0" ixz="0" iyy="0.0000001" iyz="0" izz="0.0000001"/>
+		</inertial>
+	</link>
+	<joint name="$(arg prefix)_imu_joint" type="fixed">
+		<origin xyz="0.0 0.0 0.0"/>
+		<parent link="$(arg prefix)"/>
+		<child link="$(arg prefix)_imu"/>
+		<dynamics damping="0.0" friction="0.0"/>
 	</joint>
 	<xacro:include filename="$(find riptide_description_sim)/urdf/riptide_fin.urdf.xacro"/>
@@ -35,8 +76,8 @@
 	<xacro:riptide_fin name="s" orientation="2"/>
     <!-- ROS2 control hardware interfaces -->
-    <xacro:include filename="riptide_imu.urdf.xacro"/>
-	<xacro:include filename="riptide_actuators.urdf.xacro"/>
-	<xacro:include filename="riptide_echosounder.urdf.xacro"/>
-	<xacro:include filename="riptide_pressure.urdf.xacro"/>
-	<xacro:include filename="riptide_battery.urdf.xacro"/>
+    <!-- <xacro:include filename="$(find riptide_description_sim)/urdf/riptide_imu.urdf.xacro"/> -->
+	<!-- <xacro:include filename="$(find riptide_description_sim)/urdf/riptide_actuators.urdf.xacro"/> -->
+	<!-- <xacro:include filename="$(find riptide_description_sim)/urdf/riptide_pressure.urdf.xacro"/> -->
+	<xacro:include filename="$(find riptide_description_sim)/urdf/gazebo.urdf.xacro"/>
+	<xacro:include filename="$(find riptide_description_sim)/urdf/ros2control.urdf.xacro"/>
 </robot>

File: urdf/riptide_fin.urdf.xacro (robot description, xacro)
@@ -2,5 +2,5 @@
 <robot name="$(arg prefix)" xmlns:xacro="http://www.ros.org/wiki/xacro">
     <xacro:macro name="riptide_fin" params="name orientation">
-		<xacro:property name="angle" value="${-2*orientation*pi/3 + pi/2}"/>
+		<xacro:property name="angle" value="${-2*orientation*pi/3 - pi/2}"/>
 		<link name="$(arg prefix)_${name}_fin">
 			<visual>
@@ -10,12 +10,49 @@
 				</geometry>
 			</visual>
+			<inertial>
+                <mass value="0.01" />
+                <inertia ixx="0.00001" ixy="0" ixz="0" iyy="0.00001" iyz="0" izz="0.000005" />
+            </inertial>
+			<collision>
+				<origin xyz="-0.01 0.04 0" rpy="0 0 0" />
+                <geometry>
+                    <box size="0.08 0.1 0.08" />
+                </geometry>
+            </collision>
 		</link>
-		<joint name="$(arg prefix)_${name}_fin" type="revolute">
+		<joint name="$(arg prefix)_${name}_joint" type="revolute">
 			<axis xyz="0 0 1"/>
-			<limit effort="1000.0" lower="${-pi/4}" upper="${pi/4}" velocity="0.5"/>
 			<origin rpy="${angle-pi/2} 0 0" xyz="-.35 ${.062*cos(angle)} ${.062*sin(angle)}"/>
 			<parent link="$(arg prefix)"/>
 			<child link="$(arg prefix)_${name}_fin"/>
+			<limit effort="100000.0" lower="${-pi/4}" upper="${pi/4}" velocity="0.5"/>
+			<dynamics damping="0.0" friction="0.0"/>
 		</joint>
+		<gazebo>
+			<plugin filename="ignition-gazebo-lift-drag-system" name="ignition::gazebo::systems::LiftDrag">
+				<link_name>$(arg prefix)_${name}_fin</link_name>
+				<control_joint_name>$(arg prefix)_${name}_joint</control_joint_name>
+				<air_density>1000</air_density>
+				<cla>4.13</cla>
+				<cla_stall>-1.1</cla_stall>
+				<cda>0.2</cda>
+				<cda_stall>0.03</cda_stall>
+				<alpha_stall>0.17</alpha_stall>
+				<a0>0</a0>
+				<area>0.0244</area>
+				<upward>0 1 0</upward>
+				<forward>1 0 0</forward>
+				<cp>0 0 0.05</cp>
+			</plugin>
+		</gazebo>
+		<gazebo reference="$(arg prefix)_${name}_fin">
+			<visual>
+				<material>
+                    <ambient>1. 1. 1. 0.4</ambient>
+                    <diffuse>1. 1. 1. 0.4</diffuse>
+                    <specular>1. 1. 1. 0.4</specular>
+                </material>
+			</visual>
+		</gazebo>
 	</xacro:macro>
 </robot>

Commit message: Updating riptide_description sim

File: urdf/riptide.urdf.xacro (robot description, xacro)
@@ -88,7 +88,4 @@
 	<xacro:riptide_fin name="s" orientation="2"/>
     <!-- ROS2 control hardware interfaces -->
-    <!-- <xacro:include filename="$(find riptide_description_sim)/urdf/riptide_imu.urdf.xacro"/> -->
-	<!-- <xacro:include filename="$(find riptide_description_sim)/urdf/riptide_actuators.urdf.xacro"/> -->
-	<!-- <xacro:include filename="$(find riptide_description_sim)/urdf/riptide_pressure.urdf.xacro"/> -->
 	<xacro:include filename="$(find riptide_description_sim)/urdf/gazebo.urdf.xacro"/>
 	<xacro:include filename="$(find riptide_description_sim)/urdf/ros2control.urdf.xacro"/>

File: urdf/riptide_fin.urdf.xacro (robot description, xacro)
@@ -21,11 +21,11 @@
             </collision>
 		</link>
-		<joint name="$(arg prefix)_${name}_joint" type="revolute">
+		<joint name="$(arg prefix)_${name}_joint" type="continuous">
 			<axis xyz="0 0 1"/>
 			<origin rpy="${angle-pi/2} 0 0" xyz="-.35 ${.062*cos(angle)} ${.062*sin(angle)}"/>
 			<parent link="$(arg prefix)"/>
 			<child link="$(arg prefix)_${name}_fin"/>
-			<limit effort="100000.0" lower="${-pi/4}" upper="${pi/4}" velocity="0.5"/>
-			<dynamics damping="0.0" friction="0.0"/>
+			<limit effort="1000.0" lower="${-pi/4}" upper="${pi/4}" velocity="0.5"/>
+			<dynamics damping="0.1" friction="0.1"/>
 		</joint>
 		<gazebo>

File: urdf/riptide_pressure.urdf.xacro (robot description, xacro)
@@ -3,14 +3,9 @@
     <ros2_control name="$(arg prefix)_pressure" type="sensor">
         <hardware>
-            <plugin>riptide_hardware_sim/PressureHardwareSim</plugin>
-            <param name="namespace">riptide_1</param>
-            <param name="pressure_topic">pressure</param>
-            <!-- <param name="calibration_pressure">985</param> -->
+            <plugin>ign_ros2_control/IgnitionSystem</plugin>
+            <param name="altitude_topic">/altimeter</param>
         </hardware>
-        <sensor name="$(arg prefix)_pressure">
-            <state_interface name="pressure"/>
-            <state_interface name="temperature"/>
+        <sensor name="$(arg prefix)_pressure_sensor">
             <state_interface name="depth"/>
-            <state_interface name="altitude"/>
         </sensor>
     </ros2_control>

File: urdf/ros2control.urdf.xacro (robot description, xacro)
@@ -20,5 +20,5 @@
                 <param name="max">${pi/4}</param>
                 <param name="initial_value">0.</param>
-                <param name="position_proportional_gain">1000</param>
+                <param name="position_proportional_gain">10</param>
             </command_interface>
             <state_interface name="position"/>
@@ -29,5 +29,5 @@
                 <param name="max">${pi/4}</param>
                 <param name="initial_value">0.</param>
-                <param name="position_proportional_gain">1000</param>
+                <param name="position_proportional_gain">10</param>
             </command_interface>
             <state_interface name="position"/>
@@ -38,5 +38,5 @@
                 <param name="max">${pi/4}</param>
                 <param name="initial_value">0.</param>
-                <param name="position_proportional_gain">1000</param>
+                <param name="position_proportional_gain">10</param>
             </command_interface>
             <state_interface name="position"/>
@@ -54,4 +54,7 @@
             <state_interface name="linear_acceleration.z"/>
         </sensor>
+        <sensor name="$(arg prefix)_pressure_sensor">
+            <state_interface name="depth"/>
+        </sensor>
     </ros2_control>
 </robot>

Commit message: Update

File: urdf/riptide.urdf.xacro (robot description, xacro)
@@ -11,10 +11,10 @@
 		</visual>
 		<inertial>
-			<origin xyz="0.12 0 0.14" rpy="${-pi/2} 0 ${pi}"/>
-			<mass value="9"/>
+			<origin xyz="0 0 0.14" rpy="${-pi/2} 0 ${pi}"/>
+			<mass value="13.5"/>
 			<inertia ixx="0.03675" ixy="0" ixz="0" iyy="0.8" iyz="0" izz="0.8"/>
 		</inertial>
 		<collision>
-			<origin xyz="0 0 -0.2" rpy="0 ${-pi/2} 0" />
+			<origin xyz="0 0 0" rpy="0 ${-pi/2} 0" />
 			<geometry>
 				<box size="0.12 0.12 0.95" />

Commit message: Fixing fins

File: urdf/riptide.urdf.xacro (robot description, xacro)
@@ -5,5 +5,5 @@
 	<link name="$(arg prefix)">
 		<visual>
-			<origin xyz="0.2 0 0" rpy="${-pi/2} 0 ${pi}"/>
+			<origin xyz="-0.25 0 0" rpy="${-pi/2} 0 0"/>
 			<geometry>
 				<mesh filename="package://riptide_description_sim/meshes/riptide_body.stl" scale="0.001 0.001 0.001"/>
@@ -11,5 +11,5 @@
 		</visual>
 		<inertial>
-			<origin xyz="0 0 0.14" rpy="${-pi/2} 0 ${pi}"/>
+			<origin xyz="0 0 0.06" rpy="0 0 0"/>
 			<mass value="13.5"/>
 			<inertia ixx="0.03675" ixy="0" ixz="0" iyy="0.8" iyz="0" izz="0.8"/>
@@ -47,5 +47,5 @@
 	</link>
 	<joint name="$(arg prefix)_base_link" type="fixed">
-		<origin rpy="0 0 0" xyz="-0.51 0 0"/>
+		<origin rpy="0 0 ${pi}" xyz="0 0 0"/>
 		<parent link="base_link"/>
 		<child link="$(arg prefix)"/>
@@ -54,5 +54,5 @@
 	<joint name="$(arg prefix)_thruster_joint" type="continuous">
 		<axis xyz="1 0 0"/>
-		<origin rpy="0 0 0" xyz="-0.51 0 0"/>
+		<origin rpy="0 0 ${pi}" xyz="0.46 0 0"/>
 		<parent link="$(arg prefix)"/>
 		<child link="$(arg prefix)_thruster"/>
@@ -65,7 +65,13 @@
 			<inertia ixx="0.0000001" ixy="0" ixz="0" iyy="0.0000001" iyz="0" izz="0.0000001"/>
 		</inertial>
+		<visual>
+			<origin xyz="0.0 0.0 0.0"/>
+			<geometry>
+				<box size="0.04 0.02 0.01" />
+			</geometry>
+		</visual>
 	</link>
 	<joint name="$(arg prefix)_imu_joint" type="fixed">
-		<origin xyz="0.0 0.0 0.0"/>
+		<origin rpy="0 0 ${pi}" xyz="-0.3 0.0 0.0"/>
 		<parent link="$(arg prefix)"/>
 		<child link="$(arg prefix)_imu"/>
@@ -77,7 +83,12 @@
 			<inertia ixx="0.0000001" ixy="0" ixz="0" iyy="0.0000001" iyz="0" izz="0.0000001"/>
 		</inertial>
+		<visual>
+			<geometry>
+				<cylinder radius="0.01" length="0.01"/>
+			</geometry>
+		</visual>
 	</link>
 	<joint name="$(arg prefix)_pressure_joint" type="fixed">
-		<origin xyz="0.0 0.0 0.0"/>
+		<origin rpy="0 0 ${pi}" xyz="-0.35 0.0 -0.06"/>
 		<parent link="$(arg prefix)"/>
 		<child link="$(arg prefix)_pressure"/>
@@ -85,7 +96,7 @@
 	</joint>
 	<xacro:include filename="$(find riptide_description_sim)/urdf/riptide_fin.urdf.xacro"/>
+	<xacro:riptide_fin name="p" orientation="1"/>
 	<xacro:riptide_fin name="d" orientation="0"/>
-	<xacro:riptide_fin name="p" orientation="1"/>
-	<xacro:riptide_fin name="s" orientation="2"/>
+	<xacro:riptide_fin name="s" orientation="-1"/>
     <!-- ROS2 control hardware interfaces -->
 	<xacro:include filename="$(find riptide_description_sim)/urdf/gazebo.urdf.xacro"/>

File: urdf/riptide_fin.urdf.xacro (robot description, xacro)
@@ -2,5 +2,6 @@
 <robot name="$(arg prefix)" xmlns:xacro="http://www.ros.org/wiki/xacro">
     <xacro:macro name="riptide_fin" params="name orientation">
-		<xacro:property name="angle" value="${-2*orientation*pi/3 - pi/2}"/>
+		<xacro:property name="joint_position" value="${2*orientation*pi/3 - pi/2}"/>
+		<xacro:property name="fin_angle" value="${4*orientation*pi/3 + pi}"/>
 		<link name="$(arg prefix)_${name}_fin">
 			<visual>
@@ -23,5 +24,5 @@
 		<joint name="$(arg prefix)_${name}_joint" type="continuous">
 			<axis xyz="0 0 1"/>
-			<origin rpy="${angle-pi/2} 0 0" xyz="-.35 ${.062*cos(angle)} ${.062*sin(angle)}"/>
+			<origin rpy="${fin_angle} 0 ${pi}" xyz=".3 ${.062*cos(joint_position)} ${.062*sin(joint_position)}"/>
 			<parent link="$(arg prefix)"/>
 			<child link="$(arg prefix)_${name}_fin"/>
